File: esp32controller.kicad_pcb (KiCad board)
At the start: 2 copper layers, 80 x 100 mm, 117 parts, among them J1 Conn_02x03_Odd_Even, J10 USB_B_Micro, J11 Conn_01x04_Female, J12 Conn_01x06_Female, J14 Conn_01x04, J15 Conn_01x06, J16 Conn_01x04, J17 Conn_01x04, J18 Conn_01x03, J19 Conn_01x03, J2 Conn_01x04, J20 Conn_01x03, J21 Conn_02x09_Odd_Even, J22 Conn_02x09_Odd_Even, J23 Conn_01x03, J24 Conn_01x03, J25 Conn_01x03, J26 Conn_02x09_Odd_Even, J3 Conn_02x03_Odd_Even, J4 Conn_01x04, J5 Conn_02x03_Odd_Even, J6 Conn_01x04, J7 Micro_SD_Card_Det, J8 Conn_02x03_Odd_Even, J9 Conn_01x04, Q1 Q_NPN_BEC, Q2 Q_NPN_BEC, Q3 Q_NMOS_GDS, Q4 Q_NMOS_GDS, Q5 Q_NMOS_GDS, U1 ESP32-WROOM, U2 CH340C, U3 ADS1015, U4 SX1509, U5 TPS560430, U6 TLV1117-33

Commit message: improve schematic, fix footprints
Parts:
- removed D6: LED, Diodes_SMD:D_0805
- removed J21, J22, J26: Conn_02x09_Odd_Even, Socket_Strips:Socket_Strip_Straight_2x09_Pitch2.54mm
- removed J23, J24, J25: Conn_01x03, Socket_Strips:Socket_Strip_Straight_1x03_Pitch2.54mm
- removed R37: 22.1k, Resistors_SMD:R_0603
- removed R38, R39: 1.5k, Resistors_SMD:R_1206
- removed R40: R, Resistors_SMD:R_0603
- removed R41, R42: 0, Resistors_SMD:R_0603
- removed REF***: OSHW-Symbol_8.9x8mm_SilkScreen, Symbols:OSHW-Symbol_8.9x8mm_SilkScreen
- added A5: Pololu_Breakout_A4988, Module:Pololu_Breakout-16_15.2x20.3mm, F.Cu at (261.0, 149.2)
- added C13: 100nF, Capacitor_SMD:C_0603_1608Metric, F.Cu at (256.5, 92.7)
- added C24: 100uF, Capacitor_SMD:CP_Elec_6.3x7.7, F.Cu at (217.8, 137.8)
- added C25: 100uF, Capacitor_SMD:CP_Elec_6.3x7.7, F.Cu at (234.3, 137.2)
- added C26: 100uF, Capacitor_SMD:CP_Elec_6.3x7.7, F.Cu at (250.2, 140.3)
- added C27: 100uF, Capacitor_SMD:CP_Elec_6.3x7.7, F.Cu at (267.3, 140.3)
- added C7: 100nF, Capacitor_SMD:C_0603_1608Metric, F.Cu at (97.2, 50.8)
- added D3: LED, LED_SMD:LED_0805_2012Metric, F.Cu at (82.4, 166.0)
- added J13: Conn_01x04, ESP32Controller:Socket_Strip_Straight_1x04_Pitch2.54mm_dual, F.Cu at (235.6, 170.8)
- added SW1: SW_Push, Button_Switch_SMD:SW_Push_1P1T_NO_6x6mm_H9.5mm, F.Cu at (69.2, 37.5)
- added U7: TPS560430, Package_TO_SOT_SMD:SOT-23-6, F.Cu at (84.5, 114.3)
- added U8: TLV1117-33, Package_TO_SOT_SMD:SOT-223-3_TabPin2, F.Cu at (91.4, 134.0)
- C1: value 100uF -> 100nF; footprint Capacitors_SMD:C_0805 -> Capacitor_SMD:C_0603_1608Metric
- C10: value 100uF -> NC; footprint Capacitors_SMD:CP_Elec_6.3x7.7 -> Capacitor_SMD:C_0603_1608Metric
- C11: value 10uF -> NC; footprint Capacitors_SMD:C_0805 -> Capacitor_SMD:C_0603_1608Metric
- C12, C20: value 10uF -> 100nF; footprint Capacitors_SMD:C_0805 -> Capacitor_SMD:C_0603_1608Metric
- C14, C15: footprint Capacitors_SMD:C_0603 -> Capacitor_SMD:C_0603_1608Metric
- C16: value 100n -> 100uF; footprint Capacitors_SMD:C_0603 -> Capacitor_SMD:CP_Elec_6.3x7.7
- C17: value NC -> 100nF; footprint Capacitors_SMD:C_0603 -> Capacitor_SMD:C_0603_1608Metric
- C18: value NC -> 2.2uF; footprint Capacitors_SMD:C_0603 -> Capacitor_SMD:C_0805_2012Metric
- C19: value 2.2uF -> 22uF; footprint Capacitors_SMD:C_0805 -> Capacitor_SMD:C_0805_2012Metric
- C2, C4, C5: value 100uF -> 10uF; footprint Capacitors_SMD:CP_Elec_6.3x7.7 -> Capacitor_SMD:C_0805_2012Metric
- C21: value 100uF -> 10uF; footprint Capacitors_SMD:C_0805 -> Capacitor_SMD:C_0805_2012Metric
- C22: value 0.1uF -> 10uF; footprint Capacitors_SMD:C_0603 -> Capacitor_SMD:C_0805_2012Metric
- C23: value 22uF -> 100uF; footprint Capacitors_SMD:C_0805 -> Capacitor_SMD:CP_Elec_6.3x7.7
- C3: value 1uF -> 10uF; footprint Capacitors_SMD:C_0603 -> Capacitor_SMD:C_0805_2012Metric
- C6: value 100uF -> 1uF; footprint Capacitors_SMD:CP_Elec_6.3x7.7 -> Capacitor_SMD:C_0603_1608Metric
- C8: value 100n -> 100nF; footprint Capacitors_SMD:C_0603 -> Capacitor_SMD:C_0603_1608Metric
- C9: value 1nF -> NC; footprint Capacitors_SMD:C_0603 -> Capacitor_SMD:C_0603_1608Metric
- D1, D2: footprint Diodes_SMD:D_0603 -> Diode_SMD:D_0603_1608Metric
- D4, D5: footprint Diodes_SMD:D_0805 -> LED_SMD:LED_0805_2012Metric
- F1, F2: footprint ESP32Controller:FUSE -> ESP32Controller:Fuse_0679H
- J1: value Conn_02x03_Odd_Even -> Conn_01x06; footprint Socket_Strips:Socket_Strip_Straight_2x03_Pitch2.54mm -> Connector_PinHeader_2.54mm:PinHeader_2x03_P2.54mm_Vertical
- J10: value USB_B_Micro -> Conn_01x06_Female; footprint ESP32Controller:473460001 -> ESP32Controller:KP7.62x6
- J11: value Conn_01x04_Female -> Conn_01x04; footprint ESP32Controller:KP7.62x4 -> ESP32Controller:Socket_Strip_Straight_1x04_Pitch2.54mm_dual
- J12: value Conn_01x06_Female -> Conn_01x04; footprint ESP32Controller:KP7.62x6 -> ESP32Controller:Socket_Strip_Straight_1x04_Pitch2.54mm_dual
- J14: footprint Socket_Strips:Socket_Strip_Straight_1x04_Pitch2.54mm -> ESP32Controller:Socket_Strip_Straight_1x04_Pitch2.54mm_dual
- J15: value Conn_01x06 -> Conn_01x04; footprint Socket_Strips:Socket_Strip_Straight_1x06_Pitch2.54mm -> ESP32Controller:Socket_Strip_Straight_1x04_Pitch2.54mm_dual
- J16, J17: value Conn_01x04 -> Conn_02x03_Odd_Even; footprint Socket_Strips:Socket_Strip_Straight_2x02_Pitch2.54mm -> Connector_PinHeader_2.54mm:PinHeader_2x03_P2.54mm_Vertical
- J18, J19, J20: value Conn_01x03 -> Conn_02x03_Odd_Even; footprint Socket_Strips:Socket_Strip_Straight_1x03_Pitch2.54mm -> Connector_PinHeader_2.54mm:PinHeader_2x03_P2.54mm_Vertical
- J2: value Conn_01x04 -> USB_B; footprint ESP32Controller:Socket_Strip_Straight_1x04_Pitch2.54mm_dual -> Connector_USB:USB_B_OST_USB-B1HSxx_Horizontal
- J3, J5: value Conn_02x03_Odd_Even -> Conn_01x03; footprint Socket_Strips:Socket_Strip_Straight_2x03_Pitch2.54mm -> Connector_PinHeader_2.54mm:PinHeader_1x03_P2.54mm_Vertical
- J4: value Conn_01x04 -> Conn_01x03; footprint ESP32Controller:Socket_Strip_Straight_1x04_Pitch2.54mm_dual -> Connector_PinHeader_2.54mm:PinHeader_1x03_P2.54mm_Vertical
- J6: value Conn_01x04 -> Conn_02x16_Odd_Even; footprint ESP32Controller:Socket_Strip_Straight_1x04_Pitch2.54mm_dual -> Connector_PinHeader_2.54mm:PinHeader_2x16_P2.54mm_Vertical
- J7: value Micro_SD_Card_Det -> Conn_01x04_Female; footprint ESP32Controller:microsd -> ESP32Controller:KP7.62x4; moved to F.Cu
- J8: value Conn_02x03_Odd_Even -> Conn_01x32; footprint Socket_Strips:Socket_Strip_Straight_2x03_Pitch2.54mm -> Connector_PinHeader_2.54mm:PinHeader_2x16_P2.54mm_Vertical
- J9: value Conn_01x04 -> Micro_SD_Card_Det; footprint ESP32Controller:Socket_Strip_Straight_1x04_Pitch2.54mm_dual -> ESP32Controller:microsd
- JP1: footprint Socket_Strips:Socket_Strip_Straight_1x03_Pitch2.54mm -> Connector_PinHeader_2.54mm:PinHeader_1x03_P2.54mm_Vertical
- MK1, MK2, MK3, MK4: footprint Mounting_Holes:MountingHole_3.2mm_M3 -> MountingHole:MountingHole_3.2mm_M3
- Q1, Q2: footprint TO_SOT_Packages_SMD:SOT-23 -> Package_TO_SOT_SMD:SOT-23
- Q3, Q4, Q5: footprint TO_SOT_Packages_SMD:TO-252-2 -> Package_TO_SOT_SMD:TO-252-2
- R1: value 10k -> 4.7k; footprint Resistors_SMD:R_0603 -> Resistor_SMD:R_0603_1608Metric
- R10: value 100k -> 5k; footprint Resistors_SMD:R_0603 -> Resistor_SMD:R_0603_1608Metric
- R11, R13: value 10 -> 10k; footprint Resistors_SMD:R_0603 -> Resistor_SMD:R_0603_1608Metric
- R12, R4: value 100k -> 10k; footprint Resistors_SMD:R_0603 -> Resistor_SMD:R_0603_1608Metric
- R14, R2: value 100k -> 4.7k; footprint Resistors_SMD:R_0603 -> Resistor_SMD:R_0603_1608Metric
- R15: value 5k -> 4.7k; footprint Resistors_SMD:R_0603 -> Resistor_SMD:R_0603_1608Metric
- R16: value 5k -> 2.4k; footprint Resistors_SMD:R_0603 -> Resistor_SMD:R_1206_3216Metric
- R17: value 4.7k -> 2.4k; footprint Resistors_SMD:R_0603 -> Resistor_SMD:R_1206_3216Metric
- R18: value 10k -> 10; footprint Resistors_SMD:R_0603 -> Resistor_SMD:R_0603_1608Metric
- R19: value 10k -> 100k; footprint Resistors_SMD:R_0603 -> Resistor_SMD:R_0603_1608Metric
- R20: value 4.7k -> 10; footprint Resistors_SMD:R_0603 -> Resistor_SMD:R_0603_1608Metric
- R21: value 4.7k -> 100k; footprint Resistors_SMD:R_0603 -> Resistor_SMD:R_0603_1608Metric
- R22: value 4.7k -> 88.7k; footprint Resistors_SMD:R_0603 -> Resistor_SMD:R_0603_1608Metric
- R23: value 0 -> 10; footprint Resistors_SMD:R_0603 -> Resistor_SMD:R_0603_1608Metric
- R24: value 0 -> 22.1k; footprint Resistors_SMD:R_0603 -> Resistor_SMD:R_0603_1608Metric
- R25, R32, R33, R34, R35: value 0 -> 100k; footprint Resistors_SMD:R_0603 -> Resistor_SMD:R_0603_1608Metric
- R26: value 0 -> R; footprint Resistors_SMD:R_0603 -> Resistor_SMD:R_0603_1608Metric
- R27, R28, R29, R30, R31: value 0 -> 10k; footprint Resistors_SMD:R_0603 -> Resistor_SMD:R_0603_1608Metric
- R3: value 12k -> 4.7k; footprint Resistors_SMD:R_0603 -> Resistor_SMD:R_0603_1608Metric
- R36: value 88.7k -> 100k; footprint Resistors_SMD:R_0603 -> Resistor_SMD:R_0603_1608Metric
- R5: value 12k -> 5k; footprint Resistors_SMD:R_0603 -> Resistor_SMD:R_0603_1608Metric
- R6, R8: value 100k -> 12k; footprint Resistors_SMD:R_0603 -> Resistor_SMD:R_0603_1608Metric
- R7: value 12k -> 0; footprint Resistors_SMD:R_0603 -> Resistor_SMD:R_0603_1608Metric
- R9: value 10 -> 0; footprint Resistors_SMD:R_0603 -> Resistor_SMD:R_0603_1608Metric
- U1: value ESP32-WROOM -> CH340C; footprint ESP32-footprints-Lib:ESP32-WROOM -> Package_SO:SOP-16_4.4x10.4mm_P1.27mm
- U2: value CH340C -> ESP32-WROOM; footprint Housings_SSOP:SOP-16_4.4x10.4mm_Pitch1.27mm -> ESP32-footprints-Lib:ESP32-WROOM
- U3: value ADS1015 -> 74HC595; footprint Housings_SSOP:TSSOP-10_3x3mm_Pitch0.5mm -> Package_SO:TSSOP-16_4.4x5mm_P0.65mm
- U4: value SX1509 -> 74HC595; footprint Housings_DFN_QFN:QFN-28-1EP_4x4mm_Pitch0.4mm -> Package_SO:TSSOP-16_4.4x5mm_P0.65mm
- U5: value TPS560430 -> 74HC595; footprint TO_SOT_Packages_SMD:SOT-23-6 -> Package_SO:TSSOP-16_4.4x5mm_P0.65mm
- U6: value TLV1117-33 -> 74HC595; footprint TO_SOT_Packages_SMD:SOT-223-3_TabPin2 -> Package_SO:TSSOP-16_4.4x5mm_P0.65mm
- moved J15 213.9 mm to (269.9, 169.5)
- moved J2 205.3 mm to (245.1, 35.6)
- moved J14 201.6 mm to (252.1, 169.5)
- moved C1 191.3 mm to (245.1, 55.9), turned to 0 degrees
- moved R9 189.0 mm to (250.2, 62.2), turned to 0 degrees
- moved U1 188.0 mm to (252.7, 52.1), turned to 0 degrees
- moved R35 187.1 mm to (250.8, 150.5), turned to 0 degrees
- moved R34 184.9 mm to (233.8, 150.5), turned to 0 degrees
- moved A4 183.2 mm to (244.5, 149.2)
- moved R6 180.0 mm to (250.2, 59.7), turned to 0 degrees
- moved J12 179.4 mm to (220.3, 170.8)
- moved J10 178.5 mm to (-0.64, 186.7)
- moved R8 178.4 mm to (245.1, 62.2), turned to 0 degrees
- moved J8 176.3 mm to (248.9, 73.7), turned to 0 degrees
- moved R36 175.5 mm to (267.3, 150.5), turned to 0 degrees
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Connections:
- A1 pad 15: /IO27 -> /Q1
- A1 pad 16: /IO26 -> /Q2
- A1 pad 9: /IO25 -> /Q0
- A2 pad 15: /IO33 -> /Q4
- A2 pad 16: /IO32 -> /Q5
- A2 pad 9: /IO25 -> /Q3
- A3 pad 15: /IO14 -> /Q7
- A3 pad 16: /IO12 -> /Q8
- A3 pad 9: /IO25 -> /Q6
- A4 pad 15: /E0_STEP -> /Q10
- A4 pad 16: /E0_DIR -> /Q11
- A4 pad 9: /IO25 -> /Q9
- C10 pad 1: +24V -> /IO32
- C11 pad 1: /THERM0 -> /IO33
- C12 pad 1: /THERM1 -> VCC
- C16 pad 1: VCC -> +24V
- C17 pad 1: /IO34 -> Net-(C17-Pad1)
- C17 pad 2: GND -> Net-(C17-Pad2)
- C18 pad 1: /IO35 -> +24V
- C19 pad 1: +24V -> +5V
- C2 pad 1: +24V -> /SVP
- C20 pad 1: Net-(C20-Pad1) -> VCC
- C21 pad 1: VCC -> Net-(C21-Pad1)
- C22 pad 1: Net-(C22-Pad1) -> VCC
- C22 pad 2: Net-(C22-Pad2) -> GND
- C23 pad 1: +5V -> +24V
- C3 pad 1: VCC -> /SVN
- C4 pad 1: +24V -> /SVN
- C5 pad 1: +24V -> VCC
- C6 pad 1: +24V -> VCC
- C8 pad 1: VCC -> /EN
- C9 pad 1: /EN -> /IO35
- J1 pad 1: VCC -> GND
- J1 pad 2: Net-(A1-Pad10) -> /SVP
- J1 pad 3: VCC -> GND
- J1 pad 4: Net-(A1-Pad11) -> /SVN
- J1 pad 5: VCC -> GND
- J1 pad 6: Net-(A1-Pad12) -> /IO34
- J10 pad 1: VBUS -> /HEATER_OUT
- J10 pad 2: Net-(D2-Pad1) -> +24V
- J10 pad 3: Net-(D1-Pad1) -> /FAN_OUT
- J10 pad 4: (no net) -> +24V
- J10 pad 5: GND -> /BED_OUT
- J10 pad 6: GND -> /+24V2
- J11 pad 1: Net-(F1-Pad2) -> Net-(A1-Pad3)
- J11 pad 2: GND -> Net-(A1-Pad4)
- J11 pad 3: Net-(F2-Pad2) -> Net-(A1-Pad5)
- J11 pad 4: GND -> Net-(A1-Pad6)
- J12 pad 1: /HEATER_OUT -> Net-(A2-Pad3)
- J12 pad 2: +24V -> Net-(A2-Pad4)
- J12 pad 3: /FAN_OUT -> Net-(A2-Pad5)
- J12 pad 4: +24V -> Net-(A2-Pad6)
- J14 pad 1: VCC -> Net-(A4-Pad3)
- J14 pad 2: GND -> Net-(A4-Pad4)
- J14 pad 3: /IO21 -> Net-(A4-Pad5)
- J14 pad 4: /IO22 -> Net-(A4-Pad6)
- J15 pad 1: VCC -> Net-(A5-Pad3)
- J15 pad 2: GND -> Net-(A5-Pad4)
- J15 pad 3: /IO23 -> Net-(A5-Pad5)
- J15 pad 4: /IO18 -> Net-(A5-Pad6)
- J16 pad 1: GND -> VCC
- J16 pad 2: /AIN2 -> Net-(A1-Pad10)
- J16 pad 3: GND -> VCC
- J16 pad 4: /AIN3 -> Net-(A1-Pad11)
- J17 pad 1: GND -> VCC
- J17 pad 2: /THERM0 -> Net-(A2-Pad10)
- J17 pad 3: GND -> VCC
- J17 pad 4: /THERM1 -> Net-(A2-Pad11)
- J18 pad 1: /X_MIN -> VCC
- J18 pad 2: GND -> Net-(A3-Pad10)
- J19 pad 1: /Y_MIN -> VCC
- J19 pad 2: GND -> Net-(A4-Pad10)
- J2 pad 1: Net-(A1-Pad3) -> VBUS
- J2 pad 2: Net-(A1-Pad4) -> Net-(D2-Pad1)
- J2 pad 3: Net-(A1-Pad5) -> Net-(D1-Pad1)
- J2 pad 4: Net-(A1-Pad6) -> GND
- J20 pad 1: /Z_MIN -> VCC
- J20 pad 2: GND -> Net-(A5-Pad10)
- J3 pad 1: VCC -> /IO35
- J3 pad 2: Net-(A2-Pad10) -> GND
- J4 pad 1: Net-(A2-Pad3) -> /IO32
- J4 pad 2: Net-(A2-Pad4) -> GND
- J4 pad 3: Net-(A2-Pad5) -> VCC
- J5 pad 1: VCC -> /IO33
- J5 pad 2: Net-(A3-Pad10) -> GND
- J6 pad 1: Net-(A3-Pad3) -> +24V
- J6 pad 2: Net-(A3-Pad4) -> GND
- J6 pad 3: Net-(A3-Pad5) -> VCC
- J6 pad 4: Net-(A3-Pad6) -> GND
- J7 pad 1: (no net) -> Net-(F1-Pad2)
- J7 pad 2: /IO5 -> GND
- J7 pad 3: /IO23 -> Net-(F2-Pad2)
- J7 pad 4: VCC -> GND
- J8 pad 1: VCC -> /Q0
- J8 pad 2: Net-(A4-Pad10) -> /Q1
- J8 pad 3: VCC -> /Q2
- J8 pad 4: Net-(A4-Pad11) -> /Q3
- J8 pad 5: VCC -> /Q4
- J8 pad 6: Net-(A4-Pad12) -> /Q5
- J9 pad 1: Net-(A4-Pad3) -> (no net)
- J9 pad 2: Net-(A4-Pad4) -> /IO5
- J9 pad 3: Net-(A4-Pad5) -> /IO23
- J9 pad 4: Net-(A4-Pad6) -> VCC
- JP1 pad 2: Net-(C20-Pad1) -> Net-(C21-Pad1)
- L1 pad 1: Net-(C22-Pad2) -> Net-(C17-Pad2)
- Q2 pad 3: /IO0 -> /BCLK
- R1 pad 2: /IO25 -> /SVP
- R10 pad 2: /FAN -> /HEATER
- R11 pad 1: Net-(Q4-Pad1) -> VCC
- R11 pad 2: /HEATER -> /IO35
- R12 pad 1: GND -> VCC
- R12 pad 2: /HEATER -> /IO32
- R13 pad 1: Net-(Q5-Pad1) -> VCC
- R13 pad 2: /BED -> /IO33
- R14 pad 1: GND -> VCC
- R14 pad 2: /BED -> /IO22
- R15 pad 1: GND -> VCC
- R15 pad 2: /HEATER -> /IO21
- R16 pad 1: VCC -> +24V
- R16 pad 2: /IO0 -> Net-(D3-Pad2)
- R17 pad 1: VCC -> /+24V2
- R17 pad 2: /THERM0 -> Net-(D4-Pad2)
- R18 pad 1: VCC -> Net-(Q3-Pad1)
- R18 pad 2: /IO34 -> /FAN
- R19 pad 1: VCC -> GND
- R19 pad 2: /IO35 -> /FAN
- R2 pad 1: Net-(A1-Pad10) -> VCC
- R2 pad 2: GND -> /SVN
- R20 pad 1: VCC -> Net-(Q4-Pad1)
- R20 pad 2: /THERM1 -> /HEATER
- R21 pad 1: VCC -> GND
- R21 pad 2: /IO22 -> /HEATER
- R22 pad 1: VCC -> +5V
- R22 pad 2: /IO21 -> Net-(R22-Pad2)
- R23 pad 1: /NINT -> Net-(Q5-Pad1)
- R23 pad 2: /IO0 -> /BED
- R24 pad 1: /SVP -> Net-(R22-Pad2)
- R24 pad 2: /THERM0 -> GND
- R25 pad 1: /AIN0 -> GND
- R25 pad 2: /THERM0 -> /BED
- R26 pad 1: /SVN -> VCC
- R26 pad 2: /THERM1 -> Net-(D5-Pad2)
- R27 pad 1: /AIN1 -> VCC
- R27 pad 2: /THERM1 -> /Q0
- R28 pad 1: /IO34 -> VCC
- R28 pad 2: /X_MIN -> /Q3
- R29 pad 1: /XIO0 -> VCC
- R29 pad 2: /X_MIN -> /Q6
- R3 pad 1: /DTR -> VCC
- R3 pad 2: Net-(Q1-Pad1) -> /SVN
- R30 pad 1: /IO35 -> VCC
- R30 pad 2: /Y_MIN -> /Q9
- R31 pad 1: /XIO2 -> VCC
- R31 pad 2: /Y_MIN -> /Q12
- R32 pad 1: /IO15 -> Net-(A1-Pad10)
- R32 pad 2: /Z_MIN -> GND
- R33 pad 1: /XIO4 -> Net-(A2-Pad10)
- R33 pad 2: /Z_MIN -> GND
- R34 pad 1: /IO13 -> Net-(A3-Pad10)
- R34 pad 2: /FAN -> GND
- R35 pad 1: /XIO8 -> Net-(A4-Pad10)
- R35 pad 2: /FAN -> GND
- R36 pad 1: +5V -> Net-(A5-Pad10)
- R36 pad 2: Net-(R36-Pad2) -> GND
- R4 pad 1: Net-(A2-Pad10) -> VCC
- R4 pad 2: GND -> /EN
- R5 pad 1: /RTS -> VCC
- R5 pad 2: Net-(Q2-Pad1) -> /BCLK
- R6 pad 1: Net-(A3-Pad10) -> /DTR
- R6 pad 2: GND -> Net-(Q1-Pad1)
- R7 pad 1: VCC -> /TX
- R7 pad 2: /EN -> /RXD
- R8 pad 1: Net-(A4-Pad10) -> /RTS
- R8 pad 2: GND -> Net-(Q2-Pad1)
- R9 pad 1: Net-(Q3-Pad1) -> /RX
- R9 pad 2: /FAN -> /TXD
- U1 pad 10: /IO25 -> (no net)
- U1 pad 11: /IO26 -> (no net)
- U1 pad 12: /IO27 -> (no net)
- U1 pad 13: /IO14 -> /DTR
- U1 pad 14: /IO12 -> /RTS
- U1 pad 15: GND -> (no net)
- U1 pad 16: /IO13 -> VCC
- U1 pad 2: VCC -> /TX
- U1 pad 3: /EN -> /RX
- U1 pad 4: /SVP -> VCC
- U1 pad 5: /SVN -> Net-(D1-Pad1)
- U1 pad 6: /IO34 -> Net-(D2-Pad1)
- U1 pad 7: /IO35 -> (no net)
- U1 pad 8: /IO32 -> (no net)
- U1 pad 9: /IO33 -> (no net)
- U2 pad 10: (no net) -> /IO25
- U2 pad 11: (no net) -> /IO26
- U2 pad 12: (no net) -> /FAN
- U2 pad 13: /DTR -> /HSPI_SCK
- U2 pad 14: /RTS -> /HSPI_MISO
- U2 pad 15: (no net) -> GND
- U2 pad 16: VCC -> /HSPI_MOSI
- U2 pad 2: /TX -> VCC
- U2 pad 3: /RX -> /EN
- U2 pad 4: VCC -> /SVP
- U2 pad 5: Net-(D1-Pad1) -> /SVN
- U2 pad 6: Net-(D2-Pad1) -> /IO34
- U2 pad 7: (no net) -> /IO35
- U2 pad 8: (no net) -> /IO32
- U2 pad 9: (no net) -> /IO33
- U3 pad 1: GND -> /Q1
- U3 pad 10: /IO22 -> VCC
- U3 pad 2: (no net) -> /Q2
- U3 pad 3: GND -> /Q3
- U3 pad 4: /AIN0 -> /Q4
- U3 pad 5: /AIN1 -> /Q5
- U3 pad 6: /AIN2 -> /Q6
- U3 pad 7: /AIN3 -> /Q7
- U3 pad 8: VCC -> GND
- U3 pad 9: /IO21 -> Net-(U3-Pad9)
- U4 pad 1: /XIO2 -> /Q9
- U4 pad 10: GND -> VCC
- U4 pad 11: /XOSCIO -> /BCLK
- U4 pad 12: VCC -> /IO16
- U4 pad 13: /XIO8 -> GND
- U4 pad 14: /XIO9 -> Net-(U3-Pad9)
- U4 pad 15: /XIO10 -> /Q8
- U4 pad 16: /XIO11 -> VCC
- U4 pad 2: /XIO3 -> /Q10
- U4 pad 3: GND -> /Q11
- U4 pad 4: VCC -> /Q12
- U4 pad 5: /XIO4 -> /Q13
- U4 pad 6: /XIO5 -> /Q14
- U4 pad 7: /XIO6 -> /Q15
- U4 pad 8: /XIO7 -> GND
- U4 pad 9: /NINT -> Net-(U4-Pad9)
- U5 pad 1: Net-(C22-Pad1) -> /Q17
- U5 pad 2: GND -> /Q18
- U5 pad 3: Net-(R36-Pad2) -> /Q19
- U5 pad 4: +24V -> /Q20
- U5 pad 5: +24V -> /Q21
- U5 pad 6: Net-(C22-Pad2) -> /Q22
- U6 pad 1: GND -> /Q25
- U6 pad 2: VCC -> /Q26
- U6 pad 3: Net-(C20-Pad1) -> /Q27
Routing:
- net VCC: track 396.7 -> 0.00 mm, vias 6 -> 0
- net +24V: track 187.5 -> 0.00 mm
- net GND: track 173.6 -> 0.00 mm, vias 56 -> 0
- net /IO25: track 126.7 -> 0.00 mm, vias 2 -> 0
- net /EN: track 97.6 -> 0.00 mm, vias 2 -> 0
- net /BED: track 88.0 -> 0.00 mm
- net /IO35: track 86.4 -> 0.00 mm, vias 2 -> 0
- net /IO34: track 84.5 -> 0.00 mm, vias 2 -> 0
- net /HEATER: track 74.7 -> 0.00 mm
- net VBUS: track 70.0 -> 0.00 mm, vias 1 -> 0
- net /SVN: track 69.4 -> 0.00 mm, vias 2 -> 0
- net /SVP: track 66.8 -> 0.00 mm, vias 2 -> 0
- net /FAN: track 64.5 -> 0.00 mm
- net /IO22: track 63.6 -> 0.00 mm
- net /IO21: track 60.6 -> 0.00 mm
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- removed copper zone on B.Cu, net GND
- removed copper zone on F.Cu, net GND
Other:
- board outline removed
- board text removed: "+"
- board text removed: "+5"
- board text removed: "-"
- board text removed: "AUX"
- board text removed: "E"
- board text removed: "EN"
- board text removed: "GND"
- board text removed: "I2C"
- board text removed: "Prototype R1"
- board text removed: "SPI"
- board text removed: "USB"
- board text removed: "X"
- board text removed: "X+"
- board text removed: "X-"
- board text removed: "Y"
- board text removed: "Y+"
- board text removed: "Y-"
- board text removed: "Z"
- board text removed: "Z+"
- board text removed: "Z-"

Commit message: Routed PCB
Parts:
- moved J10 232.5 mm to (186.7, 48.9), turned to 180 degrees
- moved MK1 170.7 mm to (200.7, 47.0)
- moved J7 167.2 mm to (140.3, 48.9), turned to 180 degrees
- moved MK3 140.8 mm to (106.7, 47.0)
- moved SW1 137.0 mm to (200.1, 78.0), turned to 270 degrees
- moved C8 130.2 mm to (193.6, 82.2), turned to 90 degrees
- moved J3 130.1 mm to (147.3, 95.2), turned to 90 degrees
- moved D4 127.8 mm to (137.6, 54.3)
- moved R17 127.4 mm to (137.6, 57.3), turned to 180 degrees
- moved D3 119.8 mm to (125.6, 54.3)
- moved R16 119.2 mm to (125.6, 57.3), turned to 180 degrees
- moved J4 116.5 mm to (137.2, 95.2), turned to 90 degrees
- moved JP1 114.0 mm to (173.6, 70.1), turned to 180 degrees
- moved F1 112.8 mm to (142.6, 55.8), turned to 90 degrees
- moved F2 110.6 mm to (132.6, 55.7), turned to 90 degrees
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Connections:
- C4 pad 1: /SVN -> /IO34
- J16 pad 2: Net-(A1-Pad10) -> Net-(A1-Pad12)
- J16 pad 6: Net-(A1-Pad12) -> Net-(A1-Pad10)
- J17 pad 2: Net-(A2-Pad10) -> Net-(A2-Pad12)
- J17 pad 6: Net-(A2-Pad12) -> Net-(A2-Pad10)
- J18 pad 2: Net-(A3-Pad10) -> Net-(A3-Pad12)
- J18 pad 6: Net-(A3-Pad12) -> Net-(A3-Pad10)
- J19 pad 2: Net-(A4-Pad10) -> Net-(A4-Pad12)
- J19 pad 6: Net-(A4-Pad12) -> Net-(A4-Pad10)
- J20 pad 2: Net-(A5-Pad10) -> Net-(A5-Pad12)
- J20 pad 6: Net-(A5-Pad12) -> Net-(A5-Pad10)
- R3 pad 2: /SVN -> /IO34
Routing:
- net VCC: track 0.00 -> 438.0 mm, vias 0 -> 19
- net GND: track 0.00 -> 204.9 mm, vias 0 -> 31
- net /EN: track 0.00 -> 144.5 mm, vias 0 -> 5
- net /BCLK: track 0.00 -> 129.6 mm, vias 0 -> 4
- net /HEATER: track 0.00 -> 108.4 mm, vias 0 -> 1
- net /IO16: track 0.00 -> 105.7 mm, vias 0 -> 7
- net /BED: track 0.00 -> 105.2 mm, vias 0 -> 4
- net /TXD: track 0.00 -> 93.5 mm, vias 0 -> 4
- net /RXD: track 0.00 -> 92.0 mm, vias 0 -> 2
- net /FAN: track 0.00 -> 86.7 mm, vias 0 -> 3
- net /Q3: track 0.00 -> 84.7 mm
- net /Q2: track 0.00 -> 79.8 mm, vias 0 -> 1
- net /IO17: track 0.00 -> 75.5 mm
- net /IO23: track 0.00 -> 74.9 mm, vias 0 -> 2
- net /Q1: track 0.00 -> 74.2 mm
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- added copper zone on B.Cu, net +24V
- added copper zone on F.Cu, net +24V
- added copper zone on F.Cu, net +5V
- added copper zone on B.Cu, net GND
- added copper zone on F.Cu, net GND
- added copper zone on F.Cu, net Net-(C17-Pad2)
- added copper zone on F.Cu, net VCC
Other:
- board outline added: 101.6 x 82.6 mm
- net class Default: clearance 0.2 -> 0.17; trace_width 0.25 -> 0.2; via_dia 0.8 -> 0.6
- net class power added: clearance 0.17, trace_width 0.5, via_dia 0.6, via_drill 0.4
- rule trace_clearance: 0.2 -> 0.17
- rule trace_min: 0.2 -> 0.17
- rule via_min_size: 0.4 -> 0.6
