File: esp32controller.kicad_pcb (KiCad board)
At the start: 2 copper layers, 71.1 x 101.6 mm, 136 parts, among them J1 Conn_02x03_Odd_Even, J10 Conn_01x04, J11 Micro_SD_Card_Det, J12 USB_C_Receptacle_USB2.0, J13 Conn_01x02, J14 Conn_02x11_Odd_Even, J15 Conn_02x09_Odd_Even, J16 Conn_01x01, J17 Conn_01x01, J18 Conn_01x01, J19 Conn_01x02, J2 Conn_02x03_Odd_Even, J20 Conn_01x02, J21 Conn_01x02, J22 Conn_01x06, J23 Conn_01x03, J24 Conn_01x03, J25 Conn_01x03, J3 Conn_01x04, J4 Conn_01x04, J5 Conn_02x03_Odd_Even, J6 Conn_02x03_Odd_Even, J7 Conn_01x04, J8 Conn_01x04, J9 Conn_02x03_Odd_Even, Q1 Q_NPN_BEC, Q2 Q_NPN_BEC, Q3 Q_NMOS_GDS, Q4 Q_NMOS_GDS, Q5 Q_NMOS_GDS, SW1 SW_Push, U1 74HC595, U2 74HC595, U3 ESP32-WROOM, U4 74HC595, U5 74HC595, U6 TLV1117-33, U7 TPS5430DDA, U8 CH340C

Commit message: small tweaks
Parts:
- added REF**: OSHW-Symbol_6.7x6mm_SilkScreen, Symbol:OSHW-Symbol_6.7x6mm_SilkScreen, F.Cu at (31.0, 35.3)
- moved TP14 1.25 mm to (60.5, 46.4)
Routing:
- net +3.3V: track 546.0 -> 555.1 mm, vias 11 -> 12
- net EN: track 111.5 -> 118.8 mm, vias 0 -> 2
- net RTS: track 25.4 -> 24.1 mm
Other:
- board text added: "1"
- board text added: "18"
- board text added: "2"
- board text added: "21"
- board text added: "DIR"
- board text added: "E1"
- board text added: "EN"
- board text added: "GND"
- board text added: "R2"
- board text added: "VIN"
- board text added: "VIN 10V-35V"
- board text added: "X"
- board text added: "X-"
- board text added: "Y"
- board text added: "Y-"
- board text added: "Z"
- board text added: "Z-"
- board text removed: "VIN 10V-25V"
