File: esp32controller.sch (KiCad schematic (older format))
At the start: 138 parts, among them J1 Conn_01x06, J10 Conn_01x06_Female, J11 Conn_01x04, J12 Conn_01x04, J13 Conn_01x04, J14 Conn_01x04, J15 Conn_01x04, J16 Conn_02x03_Odd_Even, J17 Conn_02x03_Odd_Even, J18 Conn_02x03_Odd_Even, J19 Conn_02x03_Odd_Even, J2 USB_B, J20 Conn_02x03_Odd_Even, J21 Conn_01x01, J22 Conn_01x01, J23 Conn_01x01, J3 Conn_01x03, J4 Conn_01x03, J5 Conn_01x03, J6 Conn_02x16_Odd_Even, J7 Conn_01x04_Female, J8 Conn_01x32, J9 Micro_SD_Card_Det, Q1 Q_NPN_BEC, Q2 Q_NPN_BEC, Q3 Q_NMOS_GDS, Q4 Q_NMOS_GDS, Q5 Q_NMOS_GDS, SW1 SW_Push, U1 CH340C, U2 ESP32-WROOM, U3 74HC595, U4 74HC595, U5 74HC595, U6 74HC595, U7 TPS560430, U8 TLV1117-33

Commit message: split schematic, update power circuit, switch to usb type c
Parts:
- removed A1, A2, A3, A4, A5: Pololu_Breakout_A4988, Module:Pololu_Breakout-16_15.2x20.3mm, symbol esp32controller-rescue:Pololu_Breakout_A4988-Driver_Motor
- removed C1, C12, C13, C14, C15, C17, C20, C7, C8: 100nF, Capacitor_SMD:C_0603_1608Metric, symbol Device:C
- removed C10, C11, C9: NC, Capacitor_SMD:C_0603_1608Metric, symbol Device:C
- removed C16: 100uF, Capacitor_SMD:CP_Elec_6.3x7.7, symbol Device:CP
- removed C18: 2.2uF, Capacitor_SMD:C_0805_2012Metric, symbol Device:C
- removed C19: 22uF, Capacitor_SMD:C_0805_2012Metric, symbol Device:C
- removed C2, C21, C22, C3, C4: 10uF, Capacitor_SMD:C_0805_2012Metric, symbol Device:C
- removed C23, C24, C25, C26, C27: 100uF, Capacitor_SMD:CP_Elec_6.3x7.7, symbol esp32controller-rescue:CP-Device
- removed C5: 10uF, Capacitor_SMD:C_0805_2012Metric, symbol esp32controller-rescue:C-Device
- removed C6: 1uF, Capacitor_SMD:C_0603_1608Metric, symbol esp32controller-rescue:C-Device
- removed D1, D2: D_TVS, Diode_SMD:D_0603_1608Metric, symbol Device:D_TVS
- removed D3, D4, D5: LED, LED_SMD:LED_0805_2012Metric, symbol Device:LED
- removed F1, F2: Fuse, ESP32Controller:Fuse_0679H, symbol Device:Fuse
- removed J1: Conn_01x06, Connector_PinHeader_2.54mm:PinHeader_2x03_P2.54mm_Vertical, symbol Connector_Generic:Conn_01x06
- removed J10: Conn_01x06_Female, ESP32Controller:KP7.62x6, symbol Connector:Conn_01x06_Female
- removed J11, J12, J13, J14, J15: Conn_01x04, ESP32Controller:Socket_Strip_Straight_1x04_Pitch2.54mm_dual, symbol esp32controller-rescue:Conn_01x04-Connector_Generic
- removed J16, J17, J18, J19, J20: Conn_02x03_Odd_Even, Connector_PinHeader_2.54mm:PinHeader_2x03_P2.54mm_Vertical, symbol esp32controller-rescue:Conn_02x03_Odd_Even-Connector_Generic
- removed J2: USB_B, Connector_USB:USB_B_OST_USB-B1HSxx_Horizontal, symbol Connector:USB_B
- removed J21, J22, J23: Conn_01x01, Connector_PinHeader_2.54mm:PinHeader_1x01_P2.54mm_Vertical, symbol Connector_Generic:Conn_01x01
- removed J3, J4, J5: Conn_01x03, Connector_PinHeader_2.54mm:PinHeader_1x03_P2.54mm_Vertical, symbol Connector_Generic:Conn_01x03
- removed J6: Conn_02x16_Odd_Even, Connector_PinHeader_2.54mm:PinHeader_2x16_P2.54mm_Vertical, symbol Connector_Generic:Conn_02x16_Odd_Even
- removed J7: Conn_01x04_Female, ESP32Controller:KP7.62x4, symbol Connector:Conn_01x04_Female
- removed J8: Conn_01x32, Connector_PinHeader_2.54mm:PinHeader_2x16_P2.54mm_Vertical, symbol Connector_Generic:Conn_01x32
- removed J9: Micro_SD_Card_Det, ESP32Controller:microsd, symbol esp32controller-rescue:Micro_SD_Card_Det-Connector
- removed JP1: Jumper_3_Open, Connector_PinHeader_2.54mm:PinHeader_1x03_P2.54mm_Vertical, symbol Jumper:Jumper_3_Open
- removed L1: 18uH, ESP32Controller:SDR0403, symbol Device:L
- removed MK1, MK2, MK3, MK4: Mounting_Hole, MountingHole:MountingHole_3.2mm_M3, symbol esp32controller-rescue:Mounting_Hole-Mechanical
- removed Q1, Q2: Q_NPN_BEC, Package_TO_SOT_SMD:SOT-23, symbol Device:Q_NPN_BEC
- removed Q3, Q4, Q5: Q_NMOS_GDS, Package_TO_SOT_SMD:TO-252-2, symbol Device:Q_NMOS_GDS
- removed R1, R14, R15, R2, R3: 4.7k, Resistor_SMD:R_0603_1608Metric, symbol Device:R
- removed R10: DNP 10k, Resistor_SMD:R_0603_1608Metric, symbol Device:R
- removed R11, R12, R13, R4, R5, R6, R8: 10k, Resistor_SMD:R_0603_1608Metric, symbol Device:R
- removed R16, R17: 2.4k, Resistor_SMD:R_1206_3216Metric, symbol Device:R
- removed R18, R20, R23: 10, Resistor_SMD:R_0603_1608Metric, symbol Device:R
- removed R19, R21, R25: 100k, Resistor_SMD:R_0603_1608Metric, symbol Device:R
- removed R22: 88.7k, Resistor_SMD:R_0603_1608Metric, symbol Device:R
- removed R24: 22.1k, Resistor_SMD:R_0603_1608Metric, symbol Device:R
- removed R26: R, Resistor_SMD:R_0603_1608Metric, symbol Device:R
- removed R27, R28, R29, R30, R31: 10k, Resistor_SMD:R_0603_1608Metric, symbol esp32controller-rescue:R-Device
- removed R32, R33, R34, R35, R36: 100k, Resistor_SMD:R_0603_1608Metric, symbol esp32controller-rescue:R-Device
- removed R37, R38, R39, R7: 0, Resistor_SMD:R_0603_1608Metric, symbol Device:R
- removed R9: 499, Resistor_SMD:R_0603_1608Metric, symbol Device:R
- removed SW1: SW_Push, Button_Switch_SMD:SW_Push_1P1T_NO_6x6mm_H9.5mm, symbol Switch:SW_Push
- removed TP1, TP10, TP11, TP12, TP13, TP14, TP15, TP16, TP17, TP2, TP3, TP4, TP5, TP6, TP7, TP8, TP9: TestPoint, TestPoint:TestPoint_Loop_D1.80mm_Drill1.0mm_Beaded, symbol Connector:TestPoint
- removed U1: CH340C, Package_SO:SOP-16_4.4x10.4mm_P1.27mm, symbol esp32controller-rescue:CH340G-ch34x
- removed U2: ESP32-WROOM, ESP32-footprints-Lib:ESP32-WROOM, symbol esp32controller-rescue:ESP32-WROOM-ESP32-footprints-Shem-Lib
- removed U3, U4, U5, U6: 74HC595, Package_SO:TSSOP-16_4.4x5mm_P0.65mm, symbol 74xx:74HC595
- removed U7: TPS560430, Package_TO_SOT_SMD:SOT-23-6, symbol esp32controller-rescue:TPS560430-ESP32Controller
- removed U8: TLV1117-33, Package_TO_SOT_SMD:SOT-223-3_TabPin2, symbol Regulator_Linear:TLV1117-33
Connections:
- net labels removed: +24V, +24V2, +5V, BCLK, BED, BED_OUT, DTR, EN, FAN, FAN_OUT, GND, HEATER, HEATER_OUT, HSPI_MISO, HSPI_MOSI, HSPI_SCK, HSPI_SS, IO0, IO12, IO13, IO14, IO15, IO16, IO17, IO18, IO19, IO2, IO21, IO22, IO23, IO25, IO26, IO27, IO32, IO33, IO34, IO35, IO4, IO5, Q0, Q1, Q10, Q11, Q12, Q13, Q14, Q15, Q16, Q17, Q18, Q19, Q2, Q20, Q21, Q22, Q23, Q24, Q25, Q26, Q27, Q28, Q29, Q3, Q30, Q31, Q4, Q5, Q6, Q7, Q8, Q9, RTS, RX, RXD, SCL, SDA, SDI, SDO, SVN, SVP, THERM0, THERM1, THERM2, TX, TXD, VBUS, VCC, VSPI_MISO, VSPI_MOSI, VSPI_SCK, VSPI_SS, WCLK, X_MIN, Y_MIN, Z_MIN
- wire segments 366 -> 1
- no-connect marks 18 -> 0
Other:
- note removed: "Buck converter 24V > 5V"
- note removed: "E0 STEPPER DRIVER"
- note removed: "E1 STEPPER DRIVER"
- note removed: "ESP32"
- note removed: "Endstops"
- note removed: "External debouncing circuit for the endstops\n(GPIO35 also doesn't contain an input pullup)"
- note removed: "I2C"
- note removed: "I2C SHIFT REGISTERS"
- note removed: "Linear regulator 5V > 3.3V"
- note removed: "MOSFETS"
- note removed: "POWER"
- note removed: "SDCard"
- note removed: "Switch buttons"
- note removed: "Thermistors / ADC Input"
- note removed: "USB TO SERIAL"
- note removed: "X STEPPER DRIVER"
- note removed: "Y STEPPER DRIVER"
- note removed: "Z STEPPER DRIVER"
