File: esp32controller.sch (KiCad schematic (older format))
At the start: 116 parts, among them J1 Conn_02x03_Odd_Even, J10 USB_B_Micro, J11 Conn_01x04_Female, J12 Conn_01x06_Female, J14 Conn_01x04, J15 Conn_01x06, J16 Conn_01x04, J17 Conn_01x04, J18 Conn_01x03, J19 Conn_01x03, J2 Conn_01x04, J20 Conn_01x03, J21 Conn_02x09_Odd_Even, J22 Conn_02x09_Odd_Even, J23 Conn_01x03, J24 Conn_01x03, J25 Conn_01x03, J26 Conn_02x09_Odd_Even, J3 Conn_02x03_Odd_Even, J4 Conn_01x04, J5 Conn_02x03_Odd_Even, J6 Conn_01x04, J7 Micro_SD_Card_Det, J8 Conn_02x03_Odd_Even, J9 Conn_01x04, Q1 Q_NPN_BEC, Q2 Q_NPN_BEC, Q3 Q_NMOS_GDS, Q4 Q_NMOS_GDS, Q5 Q_NMOS_GDS, U1 ESP32-WROOM, U2 CH340C, U3 ADS1015, U4 SX1509, U5 TPS560430, U6 TLV1117-33

Commit message: Prototype R2
Parts:
- removed A1, A2, A3, A4: Pololu_Breakout_A4988, Module:Pololu_Breakout-16_15.2x20.3mm, symbol esp32controller-rescue:Pololu_Breakout_A4988-Driver_Motor
- removed C1: 100uF, Capacitors_SMD:C_0805, symbol esp32controller-rescue:C-Device
- removed C10: 100uF, Capacitors_SMD:CP_Elec_6.3x7.7, symbol Device:CP
- removed C11, C12, C20: 10uF, Capacitors_SMD:C_0805, symbol Device:C
- removed C14, C15: 100nF, Capacitors_SMD:C_0603, symbol Device:C
- removed C16, C8: 100n, Capacitors_SMD:C_0603, symbol Device:C
- removed C17, C18: NC, Capacitors_SMD:C_0603, symbol Device:C
- removed C19: 2.2uF, Capacitors_SMD:C_0805, symbol Device:C
- removed C2, C4, C5, C6: 100uF, Capacitors_SMD:CP_Elec_6.3x7.7, symbol esp32controller-rescue:CP-Device
- removed C21: 100uF, Capacitors_SMD:C_0805, symbol Device:C
- removed C22: 0.1uF, Capacitors_SMD:C_0603, symbol Device:C
- removed C23: 22uF, Capacitors_SMD:C_0805, symbol Device:C
- removed C3: 1uF, Capacitors_SMD:C_0603, symbol esp32controller-rescue:C-Device
- removed C9: 1nF, Capacitors_SMD:C_0603, symbol Device:C
- removed D1, D2: D_TVS, Diodes_SMD:D_0603, symbol Device:D_TVS
- removed D4, D5, D6: LED, Diodes_SMD:D_0805, symbol Device:LED
- removed F1, F2: Fuse, ESP32Controller:FUSE, symbol Device:Fuse
- removed J1, J3, J5, J8: Conn_02x03_Odd_Even, Socket_Strips:Socket_Strip_Straight_2x03_Pitch2.54mm, symbol esp32controller-rescue:Conn_02x03_Odd_Even-Connector_Generic
- removed J10: USB_B_Micro, ESP32Controller:473460001, symbol Connector:USB_B_Micro
- removed J11: Conn_01x04_Female, ESP32Controller:KP7.62x4, symbol Connector:Conn_01x04_Female
- removed J12: Conn_01x06_Female, ESP32Controller:KP7.62x6, symbol Connector:Conn_01x06_Female
- removed J14: Conn_01x04, Socket_Strips:Socket_Strip_Straight_1x04_Pitch2.54mm, symbol Connector_Generic:Conn_01x04
- removed J15: Conn_01x06, Socket_Strips:Socket_Strip_Straight_1x06_Pitch2.54mm, symbol Connector_Generic:Conn_01x06
- removed J16, J17: Conn_01x04, Socket_Strips:Socket_Strip_Straight_2x02_Pitch2.54mm, symbol Connector_Generic:Conn_01x04
- removed J18, J19, J20, J23, J24, J25: Conn_01x03, Socket_Strips:Socket_Strip_Straight_1x03_Pitch2.54mm, symbol Connector_Generic:Conn_01x03
- removed J2, J4, J6, J9: Conn_01x04, ESP32Controller:Socket_Strip_Straight_1x04_Pitch2.54mm_dual, symbol esp32controller-rescue:Conn_01x04-Connector_Generic
- removed J21, J22, J26: Conn_02x09_Odd_Even, Socket_Strips:Socket_Strip_Straight_2x09_Pitch2.54mm, symbol Connector_Generic:Conn_02x09_Odd_Even
- removed J7: Micro_SD_Card_Det, ESP32Controller:microsd, symbol Connector:Micro_SD_Card_Det
- removed JP1: Jumper_3_Open, Socket_Strips:Socket_Strip_Straight_1x03_Pitch2.54mm, symbol Jumper:Jumper_3_Open
- removed L1: 18uH, ESP32Controller:SDR0403, symbol Device:L
- removed MK1, MK2, MK3, MK4: Mounting_Hole, Mounting_Holes:MountingHole_3.2mm_M3, symbol Mechanical:Mounting_Hole
- removed Q1, Q2: Q_NPN_BEC, TO_SOT_Packages_SMD:SOT-23, symbol Device:Q_NPN_BEC
- removed Q3, Q4, Q5: Q_NMOS_GDS, TO_SOT_Packages_SMD:TO-252-2, symbol Device:Q_NMOS_GDS
- removed R1: 10k, Resistors_SMD:R_0603, symbol esp32controller-rescue:R-Device
- removed R10, R12, R14: 100k, Resistors_SMD:R_0603, symbol Device:R
- removed R11, R13, R9: 10, Resistors_SMD:R_0603, symbol Device:R
- removed R15, R16: 5k, Resistors_SMD:R_0603, symbol Device:R
- removed R17, R20, R21, R22: 4.7k, Resistors_SMD:R_0603, symbol Device:R
- removed R18, R19: 10k, Resistors_SMD:R_0603, symbol Device:R
- removed R2, R4, R6, R8: 100k, Resistors_SMD:R_0603, symbol esp32controller-rescue:R-Device
- removed R23, R24, R25, R26, R27, R28, R29, R30, R31, R32, R33, R34, R35, R41, R42: 0, Resistors_SMD:R_0603, symbol Device:R
- removed R3, R5, R7: 12k, Resistors_SMD:R_0603, symbol Device:R
- removed R36: 88.7k, Resistors_SMD:R_0603, symbol Device:R
- removed R37: 22.1k, Resistors_SMD:R_0603, symbol Device:R
- removed R38, R39: 1.5k, Resistors_SMD:R_1206, symbol Device:R
- removed R40: R, Resistors_SMD:R_0603, symbol Device:R
- removed U1: ESP32-WROOM, ESP32-footprints-Lib:ESP32-WROOM, symbol ESP32-footprints-Shem-Lib:ESP32-WROOM
- removed U2: CH340C, Housings_SSOP:SOP-16_4.4x10.4mm_Pitch1.27mm, symbol ch34x:CH340G
- removed U3: ADS1015, Housings_SSOP:TSSOP-10_3x3mm_Pitch0.5mm, symbol ESP32Controller:ADS1015
- removed U4: SX1509, Housings_DFN_QFN:QFN-28-1EP_4x4mm_Pitch0.4mm, symbol ESP32Controller:SX1509
- removed U5: TPS560430, TO_SOT_Packages_SMD:SOT-23-6, symbol ESP32Controller:TPS560430
- removed U6: TLV1117-33, TO_SOT_Packages_SMD:SOT-223-3_TabPin2, symbol Regulator_Linear:TLV1117-33
Connections:
- net labels removed: +24V, +24V2, +5V, AIN0, AIN1, AIN2, AIN3, BED, BED_OUT, CLK, CMD, DTR, E0_DIR, E0_STEP, EN, FAN, FAN_OUT, GND, HEATER, HEATER_OUT, IO0, IO12, IO13, IO14, IO15, IO16, IO17, IO18, IO19, IO2, IO21, IO22, IO23, IO25, IO26, IO27, IO32, IO33, IO34, IO35, IO4, IO5, NINT, RTS, RX, RXD, SCL, SD0, SD1, SD2, SD3, SDA, SEN, SVN, SVP, THERM0, THERM1, TX, TXD, VBUS, VCC, VSPI_MISO, VSPI_MOSI, VSPI_SCK, VSPI_SS, XIO0, XIO1, XIO10, XIO11, XIO12, XIO13, XIO14, XIO15, XIO2, XIO3, XIO4, XIO5, XIO6, XIO7, XIO8, XIO9, XOSCIO, X_DIR, X_MAX, X_MIN, X_STEP, Y_DIR, Y_MAX, Y_MIN, Y_STEP, Z_DIR, Z_MAX, Z_MIN, Z_STEP
- wire segments 361 -> 1
- no-connect marks 13 -> 0
Other:
- note removed: "ADC"
- note removed: "Buck converter 24V > 5V"
- note removed: "E0 STEPPER DRIVER"
- note removed: "ESP32"
- note removed: "Endstops"
- note removed: "GPIO Expander"
- note removed: "I2C"
- note removed: "Linear regulator 5V > 3.3V"
- note removed: "MOSFETS"
- note removed: "POWER"
- note removed: "SDCard"
- note removed: "SPI"
- note removed: "Select if thermistor output goes\nto ESP32 or ADS1015"
- note removed: "Thermistors / ADC Input"
- note removed: "USB TO SERIAL"
- note removed: "X STEPPER DRIVER"
- note removed: "Y STEPPER DRIVER"
- note removed: "Z STEPPER DRIVER"
- note removed: "i2c addresses\n00 0x3e\n01 0x3f\n10 0x70\n11 0x71"
- note removed: "i2c addresses\nGND 0x48\nVDD 0x49\nSDA 0x4A\nSCL 0x4B"
- note removed: "need external pullups for 34 and 35\nthese pins can only be inputs \nand don't have pull-up/down resistors"

Commit message: Prototype R3
Changed lines of the file:
@@
 EESchema Schematic File Version 4
-LIBS:esp32controller-cache
-EELAYER 29 0
+EELAYER 30 0
 EELAYER END
 $Descr A4 11693 8268
 encoding utf-8
-Sheet 1 7
+Sheet 1 6
 Title ""
 Date ""
@@
 	750  10050 750  10250
 $Sheet
-S 7200 1650 1150 850
-U 5D75460E
-F0 "Comms" 50
-F1 "comms.sch" 50
-$EndSheet
-$Sheet
 S 6000 1650 1150 850
 U 5D7ABD98
@@
 $EndSheet
 $Sheet
-S 8400 1650 1200 850
+S 7200 1650 1200 850
 U 5DCEED1C
 F0 "Connectors" 50
