File: comms.sch (KiCad schematic (older format))
At the start: 21 parts, among them J11 Micro_SD_Card_Det, J12 USB_C_Receptacle_USB2.0, Q1 Q_NPN_BEC, Q2 Q_NPN_BEC, U8 CH340C

Commit message: finish routing
Parts:
- removed TP16, TP17: TestPoint, TestPoint:TestPoint_Pad_D1.5mm, symbol Connector:TestPoint
Changed lines of the file:
@@
 	1    0    0    -1
-$EndComp
-$Comp
-L Connector:TestPoint TP?
-U 1 1 5D770AF6
-P 9400 3450
-AR Path="/5D770AF6" Ref="TP?"  Part="1"
-AR Path="/5D75460E/5D770AF6" Ref="TP16"  Part="1"
-F 0 "TP16" H 9350 3650 50  0000 L CNN
-F 1 "TestPoint" H 9458 3477 50  0001 L CNN
-F 2 "TestPoint:TestPoint_Pad_D1.5mm" H 9600 3450 50  0001 C CNN
-F 3 "~" H 9600 3450 50  0001 C CNN
-	1    9400 3450
-	1    0    0    -1
-$EndComp
-$Comp
-L Connector:TestPoint TP?
-U 1 1 5D770AFD
-P 9400 4350
-AR Path="/5D770AFD" Ref="TP?"  Part="1"
-AR Path="/5D75460E/5D770AFD" Ref="TP17"  Part="1"
-F 0 "TP17" H 9350 4550 50  0000 L CNN
-F 1 "TestPoint" H 9458 4377 50  0001 L CNN
-F 2 "TestPoint:TestPoint_Pad_D1.5mm" H 9600 4350 50  0001 C CNN
-F 3 "~" H 9600 4350 50  0001 C CNN
-	1    9400 4350
-	-1   0    0    1
 $EndComp
 Wire Notes Line
@@
 Wire Wire Line
 	9550 3450 9400 3450
-Connection ~ 9400 3450
 Text GLabel 9550 4350 2    50   Input ~ 0
 IO0
 Wire Wire Line
 	9550 4350 9400 4350
-Connection ~ 9400 4350
 Text GLabel 8200 2900 0    50   Input ~ 0
 +3.3V

Commit message: Prototype R3
Parts:
- removed C28: 100nF, Capacitor_SMD:C_0603_1608Metric, symbol Device:C
- removed Q1, Q2: Q_NPN_BEC, Package_TO_SOT_SMD:SOT-23, symbol Device:Q_NPN_BEC
- removed R28: 0, Resistor_SMD:R_0603_1608Metric, symbol Device:R
- removed R29: 499, Resistor_SMD:R_0603_1608Metric, symbol Device:R
- removed R30, R31: 10k, Resistor_SMD:R_0603_1608Metric, symbol Device:R
- removed TP12, TP13, TP14, TP15: TestPoint, TestPoint:TestPoint_Pad_D1.5mm, symbol Connector:TestPoint
- removed U8: CH340C, Package_SO:SOP-16_4.4x10.4mm_P1.27mm, symbol esp32controller-rescue:CH340G-ch34x
- added R? (x4): 220, symbol Device:R
- added R?: 10k, symbol Device:R
Connections:
- net labels removed: DTR, EN, IO0, RTS, RX, RXD, TX, TXD
- wire segments 47 -> 27
- no-connect marks 13 -> 6
Other:
- note added: "USB"
- note removed: "USB TO SERIAL"
