File: connectors.sch (KiCad schematic (older format))
At the start: 15 parts, among them J13 Conn_01x02, J14 Conn_02x16_Odd_Even, J15 Conn_02x09_Odd_Even, J16 Conn_01x01, J17 Conn_01x01, J18 Conn_01x01, J19 Conn_01x02, J20 Conn_01x02, J21 Conn_01x02, J22 Conn_01x06, J23 Conn_01x03, J24 Conn_01x03, J25 Conn_01x03

Commit message: start R2 PCB
Parts:
- J14: value Conn_02x16_Odd_Even -> Conn_02x11_Odd_Even; footprint Connector_PinHeader_2.54mm:PinHeader_2x16_P2.54mm_Vertical -> Connector_PinHeader_2.54mm:PinHeader_2x11_P2.54mm_Vertical; symbol Connector_Generic:Conn_02x16_Odd_Even -> Connector_Generic:Conn_02x11_Odd_Even
Connections:
- net BCLK is gone; now on net HSPI_SS: J14.16 (Pin_16)
- net SDI is gone; now on net IO26: J14.19 (Pin_19)
- net WCLK is gone; now on net HSPI_MISO: J14.18 (Pin_18)
- net +3.3V: now also J14.1 (Pin_1), J14.7 (Pin_7)
- net BED: now also J14.14 (Pin_14); no longer J14.17 (Pin_17)
- net BED_OUT: now also J21.2 (Pin_2); no longer J21.1 (Pin_1)
- net EN: now also J14.22 (Pin_22); no longer J14.5 (Pin_5)
- net FAN: now also J14.20 (Pin_20); no longer J14.8 (Pin_8)
- net GND: now also J13.2 (Pin_2), J14.2 (Pin_2), J14.8 (Pin_8), J15.17 (Pin_17); no longer J13.1 (Pin_1), J15.18 (Pin_18)
- net HEATER: now also J14.13 (Pin_13); no longer J14.15 (Pin_15)
- net HSPI_MISO: no longer J14.11 (Pin_11)
- net HSPI_MOSI: now also J14.15 (Pin_15); no longer J14.12 (Pin_12)
- net HSPI_SCK: now also J14.17 (Pin_17); no longer J14.13 (Pin_13)
- net HSPI_SS: no longer J14.14 (Pin_14)
- net IO25: now also J14.21 (Pin_21); no longer J14.6 (Pin_6)
- net IO26: no longer J14.7 (Pin_7)
- net Q15: now also J15.2 (Pin_2); no longer J15.1 (Pin_1)
- net Q16: now also J15.1 (Pin_1); no longer J15.2 (Pin_2)
- net Q17: now also J15.4 (Pin_4); no longer J15.3 (Pin_3)
- net Q18: now also J15.3 (Pin_3); no longer J15.4 (Pin_4)
- net Q19: now also J15.6 (Pin_6); no longer J15.5 (Pin_5)
- net Q20: now also J15.5 (Pin_5); no longer J15.6 (Pin_6)
- net Q21: now also J15.8 (Pin_8); no longer J15.7 (Pin_7)
- net Q22: now also J15.7 (Pin_7); no longer J15.8 (Pin_8)
- net Q23: now also J15.10 (Pin_10); no longer J15.9 (Pin_9)
- net Q24: now also J15.9 (Pin_9); no longer J15.10 (Pin_10)
- net Q25: now also J15.12 (Pin_12); no longer J15.11 (Pin_11)
- net Q26: now also J15.11 (Pin_11); no longer J15.12 (Pin_12)
- net Q27: now also J15.14 (Pin_14); no longer J15.13 (Pin_13)
- net Q28: now also J15.13 (Pin_13); no longer J15.14 (Pin_14)
- net Q29: now also J15.16 (Pin_16); no longer J15.15 (Pin_15)
- net Q30: now also J15.15 (Pin_15); no longer J15.16 (Pin_16)
- net Q31: now also J15.18 (Pin_18); no longer J15.17 (Pin_17)
- net RXD: now also J14.3 (Pin_3); no longer J14.31 (Pin_31)
- net SCL: now also J14.6 (Pin_6); no longer J14.30 (Pin_30)
- net SDA: now also J14.5 (Pin_5); no longer J14.29 (Pin_29)
- net TXD: now also J14.4 (Pin_4); no longer J14.32 (Pin_32)
- net VBED_FUSED: now also J21.1 (Pin_1); no longer J21.2 (Pin_2)
- net VIN: now also J13.1 (Pin_1); no longer J13.2 (Pin_2)
- net VSPI_MISO: now also J14.9 (Pin_9); no longer J14.23 (Pin_23)
- net VSPI_MOSI: now also J14.10 (Pin_10); no longer J14.24 (Pin_24)
- net VSPI_SCK: now also J14.12 (Pin_12); no longer J14.25 (Pin_25)
- net VSPI_SS: now also J14.11 (Pin_11); no longer J14.26 (Pin_26)
Other:
- moved on the sheet: J15

Commit message: Prototype R3
Parts:
- removed J13: Conn_01x02, ESP32-footprints-Lib:TERM_2-WAY_6.35mm, symbol Connector_Generic:Conn_01x02
- removed J14: Conn_02x11_Odd_Even, Connector_PinHeader_2.54mm:PinHeader_2x11_P2.54mm_Vertical, symbol Connector_Generic:Conn_02x11_Odd_Even
- removed J15: Conn_02x09_Odd_Even, Connector_PinHeader_2.54mm:PinHeader_2x09_P2.54mm_Vertical, symbol Connector_Generic:Conn_02x09_Odd_Even
- removed J16, J17, J18: Conn_01x01, Connector_PinHeader_2.54mm:PinHeader_1x01_P2.54mm_Vertical, symbol Connector_Generic:Conn_01x01
- removed J22: Conn_01x06, Connector_PinHeader_2.54mm:PinHeader_2x03_P2.54mm_Vertical, symbol Connector_Generic:Conn_01x06
- added C33: 100nF, Capacitor_SMD:C_0603_1608Metric, symbol Device:C
- added D5, D6: D_TVS, Diode_SMD:D_SOD-523, symbol Device:D_TVS
- added J41: T0, Connector_JST:JST_XH_B2B-XH-A_1x02_P2.50mm_Vertical, symbol Connector_Generic:Conn_01x02
- added J42: HSPI, Connector_IDC:IDC-Header_2x03_P2.54mm_Vertical, symbol Connector_Generic:Conn_02x03_Odd_Even
- added J43: I2S EXT, Connector_JST:JST_XH_B4B-XH-A_1x04_P2.50mm_Vertical, symbol Connector_Generic:Conn_01x04
- added J44: UART, Connector_IDC:IDC-Header_2x04_P2.54mm_Vertical, symbol Connector_Generic:Conn_02x04_Odd_Even
- added J46: T1, Connector_JST:JST_XH_B2B-XH-A_1x02_P2.50mm_Vertical, symbol Connector_Generic:Conn_01x02
- added J47: VIN, ESP32-footprints-Lib:TERM_2-WAY_6.35mm, symbol Connector_Generic:Conn_01x02
- added J48: T2, Connector_JST:JST_XH_B2B-XH-A_1x02_P2.50mm_Vertical, symbol Connector_Generic:Conn_01x02
- added J50: VSPI, Connector_IDC:IDC-Header_2x03_P2.54mm_Vertical, symbol Connector_Generic:Conn_02x03_Odd_Even
- added J51: T3, Connector_JST:JST_XH_B2B-XH-A_1x02_P2.50mm_Vertical, symbol Connector_Generic:Conn_01x02
- added J53: I2C, Connector_JST:JST_XH_B4B-XH-A_1x04_P2.50mm_Vertical, symbol Connector_Generic:Conn_01x04
- added J54: T4, Connector_JST:JST_XH_B2B-XH-A_1x02_P2.50mm_Vertical, symbol Connector_Generic:Conn_01x02
- added J55: BLTOUCH, Connector_PinHeader_2.54mm:PinHeader_1x03_P2.54mm_Vertical, symbol Connector_Generic:Conn_01x03
- added J56: EXT, Connector_IDC:IDC-Header_2x03_P2.54mm_Vertical, symbol Connector_Generic:Conn_02x03_Odd_Even
- added J57: Conn_01x02, Connector_PinHeader_2.54mm:PinHeader_1x02_P2.54mm_Vertical, symbol Connector_Generic:Conn_01x02
- added J66: MOS3, TerminalBlock:TerminalBlock_bornier-2_P5.08mm, symbol Connector_Generic:Conn_01x02
- added J67: USB_C_Receptacle_USB2.0, ESP32Controller:USB_C, symbol Connector:USB_C_Receptacle_USB2.0
- added J68: Micro_SD_Card_Det, ESP32Controller:microsd, symbol esp32controller-rescue:Micro_SD_Card_Det-Connector
- added J69: MOS4, TerminalBlock:TerminalBlock_bornier-2_P5.08mm, symbol Connector_Generic:Conn_01x02
- added J70: VBED, ESP32-footprints-Lib:TERM_2-WAY_6.35mm, symbol Connector_Generic:Conn_01x02
- added R41: 10k, Resistor_SMD:R_0603_1608Metric, symbol Device:R
- added R42, R43: 5.1k, Resistor_SMD:R_0603_1608Metric, symbol Device:R
- added R44, R45, R46, R47: 220, Resistor_SMD:R_0603_1608Metric, symbol Device:R
- F1, F2: footprint ESP32Controller:Fuse_0679H -> ESP32Controller:Fuse_holder_0679H
- J45: renamed from J23; value Conn_01x03 -> S0; footprint Connector_PinHeader_2.54mm:PinHeader_1x03_P2.54mm_Vertical -> Connector_JST:JST_XH_B3B-XH-A_1x03_P2.50mm_Vertical
- J49: renamed from J24; value Conn_01x03 -> S1; footprint Connector_PinHeader_2.54mm:PinHeader_1x03_P2.54mm_Vertical -> Connector_JST:JST_XH_B3B-XH-A_1x03_P2.50mm_Vertical
- J52: renamed from J25; value Conn_01x03 -> S2; footprint Connector_PinHeader_2.54mm:PinHeader_1x03_P2.54mm_Vertical -> Connector_JST:JST_XH_B3B-XH-A_1x03_P2.50mm_Vertical
- J59: renamed from J19; value Conn_01x02 -> MOS0; footprint TerminalBlock_4Ucon:TerminalBlock_4Ucon_1x02_P3.50mm_Horizontal -> ESP32-footprints-Lib:TERM_2-WAY_6.35mm
- J61: renamed from J20; value Conn_01x02 -> MOS1; footprint TerminalBlock_4Ucon:TerminalBlock_4Ucon_1x02_P3.50mm_Horizontal -> TerminalBlock:TerminalBlock_bornier-2_P5.08mm
- J64: renamed from J21; value Conn_01x02 -> MOS2; footprint ESP32-footprints-Lib:TERM_2-WAY_6.35mm -> TerminalBlock:TerminalBlock_bornier-2_P5.08mm
Connections:
- net HEATER_OUT is gone; now on net VIN_FUSED: J61.1 (Pin_1)
- net +3.3V: now also C33.1, J42.2 (Pin_2), J43.1 (Pin_1), J44.7 (Pin_7), J50.2 (Pin_2), J53.1 (Pin_1), J56.5 (Pin_5), J68.4 (VDD), R41.1
- net EN: now also J44.6 (Pin_6)
- net GND: now also C33.2, D5.2 (A2), D6.2 (A2), J41.1 (Pin_1), J42.6 (Pin_6), J43.4 (Pin_4), J44.8 (Pin_8), J46.1 (Pin_1), J47.1 (Pin_1), J48.1 (Pin_1), J50.6 (Pin_6), J51.1 (Pin_1), J53.4 (Pin_4), J54.1 (Pin_1), J55.1 (Pin_1), J56.6 (Pin_6), J57.2 (Pin_2), J67.A1 (GND), J67.A12 (GND), J67.B1 (GND), J67.B12 (GND), J67.S1 (SHIELD), J68.10 (DET_A), J68.11 (SHIELD), J68.6 (VSS), J70.1 (Pin_1), R42.1, R43.1
- net HSPI_MISO: now also J42.1 (Pin_1)
- net HSPI_MOSI: now also J42.4 (Pin_4)
- net Q15: now also J43.3 (Pin_3)
- net Q31: now also J43.2 (Pin_2)
- net SCL: now also J53.3 (Pin_3)
- net SDA: now also J53.2 (Pin_2)
- net THERM0: now also J41.2 (Pin_2)
- net THERM1: now also J46.2 (Pin_2)
- net THERM2: now also J48.2 (Pin_2)
- net VBED_FUSED: now also J59.2 (Pin_2); no longer J64.1 (Pin_1)
- net VIN: now also J47.2 (Pin_2); no longer F2.2
- net VIN_FUSED: now also J64.1 (Pin_1), J66.1 (Pin_1), J69.1 (Pin_1); no longer J59.2 (Pin_2), J61.2 (Pin_2)
- net VSPI_MISO: now also J50.1 (Pin_1), R47.1
- net VSPI_MOSI: now also J50.4 (Pin_4), R45.1
- net BED_OUT renamed MOS2_OUT
- net FAN_OUT renamed MOS0_OUT
- net X_MIN renamed S0_MIN
- net Y_MIN renamed S1_MIN
- net Z_MIN renamed S2_MIN
- new net: J68.2 (DAT3/CD), R44.2
- new net: J68.3 (CMD), R41.2, R45.2
- new net: J68.5 (CLK), R46.2
- new net: J68.7 (DAT0), R47.2
- new net: J67.A5 (CC1), R42.2
- new net: J67.B5 (CC2), R43.2
- new net +5V: J55.2 (Pin_2)
- new net HSPI_CLK: J42.3 (Pin_3)
- new net HSPI_CS: J42.5 (Pin_5)
- new net IO0: J44.5 (Pin_5), J55.3 (Pin_3)
- new net IO38: J56.3 (Pin_3)
- new net IO39: J56.4 (Pin_4)
- new net IO45: J56.1 (Pin_1)
- new net IO46: J56.2 (Pin_2), J57.1 (Pin_1)
- new net MOS1_OUT: J61.2 (Pin_2)
- new net MOS3_OUT: J66.2 (Pin_2)
- new net MOS4_OUT: J69.2 (Pin_2)
- new net RX0: J44.4 (Pin_4)
- new net RX1: J44.2 (Pin_2)
- new net THERM3: J51.2 (Pin_2)
- new net THERM4: J54.2 (Pin_2)
- new net TX0: J44.3 (Pin_3)
- new net TX1: J44.1 (Pin_1)
- new net USB_D+: D5.1 (A1), J67.A6 (D+), J67.B6 (D+)
- new net USB_D-: D6.1 (A1), J67.A7 (D-), J67.B7 (D-)
- new net VBED: F2.2, J70.2 (Pin_2)
- new net VBUS: J67.A4 (VBUS), J67.A9 (VBUS), J67.B4 (VBUS), J67.B9 (VBUS)
- new net VSPI_CLK: J50.3 (Pin_3), R46.1
- new net VSPI_CS: J50.5 (Pin_5), R44.1
- no-connect marks 0 -> 5
Other:
- note added: "BLTOUCH"
- note added: "EXT"
- note added: "I2C"
- note added: "SDCard"
- note added: "SPI"
- note added: "UART"
- note added: "USB"
- note removed: "ESP32 breakout pins"
- note removed: "Mosfet external inputs"
- moved on the sheet: F1, F2, J59, J61, J64
