File: mosfets.sch (KiCad schematic (older format))
At the start: 12 parts, among them Q3 Q_NMOS_GDS, Q4 Q_NMOS_GDS, Q5 Q_NMOS_GDS

Commit message: Prototype R3
Parts:
- added Q4, Q5: Q_NMOS_GDS, Package_TO_SOT_SMD:TO-252-2, symbol Device:Q_NMOS_GDS
- added R35, R38: 0, Resistor_SMD:R_0603_1608Metric, symbol Device:R
- added R36, R39: 10, Resistor_SMD:R_0603_1608Metric, symbol Device:R
- added R37, R40: 100k, Resistor_SMD:R_0603_1608Metric, symbol Device:R
- renumbered Q3 to Q1, Q4 to Q2, Q5 to Q3, R32 to R26, R35 to R27, R36 to R28, R33 to R29, R37 to R30, R38 to R31, R34 to R32, R39 to R33, R40 to R34
Connections:
- net GND: now also Q4.3 (S), Q5.3 (S), R37.1, R40.1
- net BED renamed MOS2
- net BED_IN renamed MOS2_IN
- net BED_OUT renamed MOS2_OUT
- net FAN renamed MOS0
- net FAN_IN renamed MOS0_IN
- net FAN_OUT renamed MOS0_OUT
- net HEATER renamed MOS1
- net HEATER_IN renamed MOS1_IN
- net HEATER_OUT renamed MOS1_OUT
- new net: Q4.1 (G), R36.1
- new net: Q5.1 (G), R39.1
- new net MOS3: R35.2
- new net MOS3_IN: R35.1, R36.2, R37.2
- new net MOS3_OUT: Q4.2 (D)
- new net MOS4: R38.2
- new net MOS4_IN: R38.1, R39.2, R40.2
- new net MOS4_OUT: Q5.2 (D)
Other:
- moved on the sheet: Q1, Q2, Q3, R26, R27, R28, R29, R30, R31, R32, R33, R34
