File: power.sch (KiCad schematic (older format))
At the start: 22 parts, among them U6 TLV1117-33, U7 TPS5430DDA

Commit message: Prototype R3
Parts:
- removed C15, C17: 4.7uF, Capacitor_SMD:C_0805_2012Metric, symbol Device:C
- removed C19: 100uF, Capacitor_SMD:CP_Elec_6.3x7.7, symbol Device:CP
- removed C20: 10nF, Capacitor_SMD:C_0603_1608Metric, symbol Device:C
- removed C21: 220uF, Capacitor_SMD:C_1210_3225Metric, symbol Device:CP1_Small
- removed D3: LED, LED_SMD:LED_0805_2012Metric, symbol Device:LED
- removed D4: B340A, Diode_SMD:D_SMA, symbol Device:D_Schottky_Small
- removed R13: 2.4k, Resistor_SMD:R_1206_3216Metric, symbol Device:R
- removed R14: 10k, Resistor_SMD:R_0603_1608Metric, symbol Device:R
- removed R15: 3.24k, Resistor_SMD:R_0603_1608Metric, symbol Device:R
- removed TP10, TP11, TP8, TP9: TestPoint, TestPoint:TestPoint_Pad_D1.5mm, symbol Connector:TestPoint
- removed U7: TPS5430DDA, Package_SO:TI_SO-PowerPAD-8_ThermalVias, symbol Regulator_Switching:TPS5430DDA
- added C18: 470uF/35V, Capacitor_SMD:CP_Elec_10x10, symbol Device:CP1_Small
- added C19: 4.7uF/35V, Capacitor_SMD:C_0805_2012Metric, symbol Device:C
- added C20: 220uF/35V, Capacitor_SMD:C_1210_3225Metric, symbol Device:CP1_Small
- added D1: B340A, Diode_SMD:D_SMA, symbol Device:D_Schottky_Small
- added U6: XL1509, Package_SO:SOIC-8_3.9x4.9mm_P1.27mm, symbol ESP32Controller:XL1509
- D2: renamed from D1; footprint Diode_SMD:D_0603_1608Metric -> Diode_SMD:D_SOD-323_HandSoldering
- L1: value 22uH -> 68uH
- renumbered C16 to C21, C18 to C22, D2 to D4, R12 to R15, U6 to U7
Connections:
- net +5V: now also C20.1, U6.3 (FB)
- net GND: now also C18.2, C19.2, C20.2, D1.2 (A), U6.5 (GND), U6.6 (GND), U6.7 (GND), U6.8 (GND)
- net VIN_FUSED: now also C18.1, C19.1, U6.1 (VIN)
- net at L1.1: now also D1.1 (K), U6.2 (OUT)
Other:
- note added: "Buck converter\n10V-35V Input > 5V 2A Output"
- note removed: "Buck converter\n10V-35V Input > 5V 3A Output"
- note removed: "Power Cap.\n"
